Commit message: reorgnize structure

File: pbrs-humanoid/resources/robots/mit_humanoid/mit_humanoid_fixed_arms.urdf (robot description, URDF)
Before this commit: robot humanoid, 21 links, 20 joints
Links:
- link left_foot: mass  0.279583 -> 0.279583
- link left_hip_yaw: mass  0.842752 -> 0.842752
- link right_foot: mass  0.279583 -> 0.279583
- link right_hip_yaw: mass  0.842752 -> 0.842752
